Commit message: modified_aiw

File: ffw_description/gazebo/ffw_bg2_rev4_follower/ffw_bg2_follower.gazebo.xacro (robot description, xacro)
@@ -78,3 +78,58 @@
   <xacro:SimpleTransmission trans="l_tran_l2" joint="l_rh_l2" actuator="l_actuator4" />
   </xacro:macro>
+  <!-- Simulation RGB cameras. use_cam:=true -->
+  <xacro:macro name="ffw_bg2_follower_gazebo_cameras">
+    <gazebo reference="zed_left_camera_frame">
+      <sensor name="head_camera" type="camera">
+        <always_on>true</always_on>
+        <update_rate>30</update_rate>
+        <topic>head_camera/image</topic>
+        <gz_frame_id>zed_left_camera_optical_frame</gz_frame_id>
+        <camera>
+          <horizontal_fov>1.7802</horizontal_fov>
+          <image><width>672</width><height>376</height><format>R8G8B8</format></image>
+          <clip><near>0.05</near><far>10</far></clip>
+        </camera>
+      </sensor>
+    </gazebo>
+    <link name="camera_left_color_optical_frame"/>
+    <joint name="camera_left_color_optical_joint" type="fixed">
+      <parent link="camera_left_link"/>
+      <child link="camera_left_color_optical_frame"/>
+      <origin xyz="0 0 0" rpy="-1.5707963 0 -1.5707963"/>
+    </joint>
+    <gazebo reference="camera_left_link">
+      <sensor name="wrist_left_camera" type="camera">
+        <always_on>true</always_on>
+        <update_rate>30</update_rate>
+        <topic>wrist_left_camera/image</topic>
+        <gz_frame_id>camera_left_color_optical_frame</gz_frame_id>
+        <camera>
+          <horizontal_fov>1.5184</horizontal_fov>
+          <image><width>424</width><height>240</height><format>R8G8B8</format></image>
+          <!-- near 0.01 keeps the gripper fingers right in front of the lens visible. -->
+          <clip><near>0.01</near><far>5</far></clip>
+        </camera>
+      </sensor>
+    </gazebo>
+    <link name="camera_right_color_optical_frame"/>
+    <joint name="camera_right_color_optical_joint" type="fixed">
+      <parent link="camera_right_link"/>
+      <child link="camera_right_color_optical_frame"/>
+      <origin xyz="0 0 0" rpy="-1.5707963 0 -1.5707963"/>
+    </joint>
+    <gazebo reference="camera_right_link">
+      <sensor name="wrist_right_camera" type="camera">
+        <always_on>true</always_on>
+        <update_rate>30</update_rate>
+        <topic>wrist_right_camera/image</topic>
+        <gz_frame_id>camera_right_color_optical_frame</gz_frame_id>
+        <camera>
+          <horizontal_fov>1.5184</horizontal_fov>
+          <image><width>424</width><height>240</height><format>R8G8B8</format></image>
+          <clip><near>0.01</near><far>5</far></clip>
+        </camera>
+      </sensor>
+    </gazebo>
+  </xacro:macro>
 </robot>

File: ffw_description/gazebo/ffw_sg2_rev1_follower/ffw_sg2_follower.gazebo.xacro (robot description, xacro)
@@ -43,14 +43,14 @@
   <xacro:Link reference="arm_l_link6"/>
   <xacro:Link reference="arm_l_link7"/>
-  <xacro:Link reference="r_rh_p12_rn_base"/>
-  <xacro:Link reference="r_rh_p12_rn_r1"/>
-  <xacro:Link reference="r_rh_p12_rn_r2"/>
-  <xacro:Link reference="r_rh_p12_rn_l1"/>
-  <xacro:Link reference="r_rh_p12_rn_l2"/>
-  <xacro:Link reference="l_rh_p12_rn_base"/>
-  <xacro:Link reference="l_rh_p12_rn_r1"/>
-  <xacro:Link reference="l_rh_p12_rn_r2"/>
-  <xacro:Link reference="l_rh_p12_rn_l1"/>
-  <xacro:Link reference="l_rh_p12_rn_l2"/>
+  <xacro:Link reference="gripper_r_rh_p12_rn_base"/>
+  <xacro:Link reference="gripper_r_rh_p12_rn_r1"/>
+  <xacro:Link reference="gripper_r_rh_p12_rn_r2"/>
+  <xacro:Link reference="gripper_r_rh_p12_rn_l1"/>
+  <xacro:Link reference="gripper_r_rh_p12_rn_l2"/>
+  <xacro:Link reference="gripper_l_rh_p12_rn_base"/>
+  <xacro:Link reference="gripper_l_rh_p12_rn_r1"/>
+  <xacro:Link reference="gripper_l_rh_p12_rn_r2"/>
+  <xacro:Link reference="gripper_l_rh_p12_rn_l1"/>
+  <xacro:Link reference="gripper_l_rh_p12_rn_l2"/>
   <xacro:SimpleTransmission trans="lift_trans" joint="lift_joint" actuator="lift_actuator"/>
   <xacro:SimpleTransmission trans="head_trans1" joint="head_joint1" actuator="head_actuator1"/>
@@ -140,3 +140,58 @@
   </gazebo>
   </xacro:macro>
+  <!-- Simulation RGB cameras. use_cam:=true -->
+  <xacro:macro name="ffw_sg2_follower_gazebo_cameras">
+    <gazebo reference="zed_left_camera_frame">
+      <sensor name="head_camera" type="camera">
+        <always_on>true</always_on>
+        <update_rate>30</update_rate>
+        <topic>head_camera/image</topic>
+        <gz_frame_id>zed_left_camera_optical_frame</gz_frame_id>
+        <camera>
+          <horizontal_fov>1.7802</horizontal_fov>
+          <image><width>672</width><height>376</height><format>R8G8B8</format></image>
+          <clip><near>0.05</near><far>10</far></clip>
+        </camera>
+      </sensor>
+    </gazebo>
+    <link name="camera_left_color_optical_frame"/>
+    <joint name="camera_left_color_optical_joint" type="fixed">
+      <parent link="camera_left_link"/>
+      <child link="camera_left_color_optical_frame"/>
+      <origin xyz="0 0 0" rpy="-1.5707963 0 -1.5707963"/>
+    </joint>
+    <gazebo reference="camera_left_link">
+      <sensor name="wrist_left_camera" type="camera">
+        <always_on>true</always_on>
+        <update_rate>30</update_rate>
+        <topic>wrist_left_camera/image</topic>
+        <gz_frame_id>camera_left_color_optical_frame</gz_frame_id>
+        <camera>
+          <horizontal_fov>1.5184</horizontal_fov>
+          <image><width>424</width><height>240</height><format>R8G8B8</format></image>
+          <!-- near 0.01 keeps the gripper fingers right in front of the lens visible. -->
+          <clip><near>0.01</near><far>5</far></clip>
+        </camera>
+      </sensor>
+    </gazebo>
+    <link name="camera_right_color_optical_frame"/>
+    <joint name="camera_right_color_optical_joint" type="fixed">
+      <parent link="camera_right_link"/>
+      <child link="camera_right_color_optical_frame"/>
+      <origin xyz="0 0 0" rpy="-1.5707963 0 -1.5707963"/>
+    </joint>
+    <gazebo reference="camera_right_link">
+      <sensor name="wrist_right_camera" type="camera">
+        <always_on>true</always_on>
+        <update_rate>30</update_rate>
+        <topic>wrist_right_camera/image</topic>
+        <gz_frame_id>camera_right_color_optical_frame</gz_frame_id>
+        <camera>
+          <horizontal_fov>1.5184</horizontal_fov>
+          <image><width>424</width><height>240</height><format>R8G8B8</format></image>
+          <clip><near>0.01</near><far>5</far></clip>
+        </camera>
+      </sensor>
+    </gazebo>
+  </xacro:macro>
 </robot>

File: ffw_description/ros2_control/ffw_bg2_rev4_follower/ffw_bg2_follower.ros2_control.xacro (robot description, xacro)
@@ -79,4 +79,18 @@
         <state_interface name="effort"/>
       </joint>
+      <xacro:if value="$(arg use_sim)">
+        <joint name="gripper_r_joint2">
+          <state_interface name="position"/>
+          <state_interface name="velocity"/>
+        </joint>
+        <joint name="gripper_r_joint3">
+          <state_interface name="position"/>
+          <state_interface name="velocity"/>
+        </joint>
+        <joint name="gripper_r_joint4">
+          <state_interface name="position"/>
+          <state_interface name="velocity"/>
+        </joint>
+      </xacro:if>
       <joint name="arm_l_joint1">
         <command_interface name="position"/>
@@ -127,4 +141,18 @@
         <state_interface name="effort"/>
       </joint>
+      <xacro:if value="$(arg use_sim)">
+        <joint name="gripper_l_joint2">
+          <state_interface name="position"/>
+          <state_interface name="velocity"/>
+        </joint>
+        <joint name="gripper_l_joint3">
+          <state_interface name="position"/>
+          <state_interface name="velocity"/>
+        </joint>
+        <joint name="gripper_l_joint4">
+          <state_interface name="position"/>
+          <state_interface name="velocity"/>
+        </joint>
+      </xacro:if>
       <joint name="lift_joint">
         <command_interface name="position"/>

File: ffw_description/ros2_control/ffw_sg2_rev1_follower/ffw_sg2_follower.ros2_control.xacro (robot description, xacro)
@@ -79,4 +79,18 @@
         <state_interface name="effort"/>
       </joint>
+      <xacro:if value="$(arg use_sim)">
+        <joint name="gripper_r_joint2">
+          <state_interface name="position"/>
+          <state_interface name="velocity"/>
+        </joint>
+        <joint name="gripper_r_joint3">
+          <state_interface name="position"/>
+          <state_interface name="velocity"/>
+        </joint>
+        <joint name="gripper_r_joint4">
+          <state_interface name="position"/>
+          <state_interface name="velocity"/>
+        </joint>
+      </xacro:if>
       <joint name="arm_l_joint1">
         <command_interface name="position"/>
@@ -127,4 +141,18 @@
         <state_interface name="effort"/>
       </joint>
+      <xacro:if value="$(arg use_sim)">
+        <joint name="gripper_l_joint2">
+          <state_interface name="position"/>
+          <state_interface name="velocity"/>
+        </joint>
+        <joint name="gripper_l_joint3">
+          <state_interface name="position"/>
+          <state_interface name="velocity"/>
+        </joint>
+        <joint name="gripper_l_joint4">
+          <state_interface name="position"/>
+          <state_interface name="velocity"/>
+        </joint>
+      </xacro:if>
       <joint name="lift_joint">
         <command_interface name="position"/>

File: ffw_description/urdf/ffw_bg2_rev4_follower/ffw_bg2_follower.urdf.xacro (robot description, xacro)
@@ -9,4 +9,5 @@
   <xacro:arg name="model" default="ffw_bg2_rev4_follower" />
   <xacro:arg name="ros2_control_type" default="ffw_bg2_follower" />
+  <xacro:arg name="use_cam" default="false" />
   <xacro:include filename="$(find ffw_description)/urdf/common/follower/ffw_follower_body.xacro" />
   <xacro:include filename="$(find ffw_description)/urdf/common/rh_p12_rn_a/rh_p12_rn_a.urdf.xacro" />
@@ -93,3 +94,6 @@
       </plugin>
   </gazebo>
+  <xacro:if value="${'$(arg use_sim)' == 'true' and '$(arg use_cam)' == 'true'}">
+    <xacro:ffw_bg2_follower_gazebo_cameras/>
+  </xacro:if>
 </robot>

File: ffw_description/urdf/ffw_sg2_rev1_follower/ffw_sg2_follower.urdf.xacro (robot description, xacro)
@@ -9,4 +9,5 @@
   <xacro:arg name="model" default="ffw_sg2_rev1_follower" />
   <xacro:arg name="ros2_control_type" default="ffw_sg2_follower" />
+  <xacro:arg name="use_cam" default="false" />
   <xacro:include filename="$(find ffw_description)/urdf/common/follower/ffw_follower_body.xacro" />
   <xacro:include filename="$(find ffw_description)/urdf/common/rh_p12_rn_a/rh_p12_rn_a.urdf.xacro" />
@@ -376,3 +377,6 @@
       </plugin>
   </gazebo>
+  <xacro:if value="${'$(arg use_sim)' == 'true' and '$(arg use_cam)' == 'true'}">
+    <xacro:ffw_sg2_follower_gazebo_cameras/>
+  </xacro:if>
 </robot>
